File: vehicle/mkvi/hardware/charging-cart/J1772/CAN_CONTROLLER.kicad_sch (KiCad schematic)
At the start: 11 parts, among them J4 CONN_01x02

Commit message: Updating branch.
Parts:
- C10, C11, C9: value 0.1uF -> C_0.1uF; footprint OEM:C_0603 -> footprints:C_0603_1608Metric; symbol OEM:0u1F -> formula:C_0.1uF; DKPN 1276-1935-2-ND -> (none); MFN Samsung Electro-Mechanics -> DK; MPN CL10B104KB8NNWC -> 478-3352-1-ND; NewDesigns YES -> (none); Package 0603 -> (none); PurchasingLink (none) -> https://www.digikey.com/products/en?keywords=478-3352-1-ND; Stocked Reel -> (none); Style SMD -> (none)
- C12, C13: footprint OEM:C_0603 -> footprints:C_0603_1608Metric; symbol OEM:30pF -> formula:C_30pF; DKPN 738-CML0603C0G300JT50VDKR-ND -> (none); MFN Stackpole Electronics -> DK; MPN CML0603C0G300JT50V -> 1276-1130-1-ND; NewDesigns YES -> (none); Package 0603 -> (none); PurchasingLink (none) -> https://www.digikey.com/product-detail/en/samsung-electro-m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; Stocked Digi-Reel -> (none); Style SMD -> (none)
- J4: symbol OEM:CONN_01x02 -> formula:CONN_01x02; DKPN 2057-PH1-02-UA-ND -> (none); MFN Adam Tech -> DK; MPN PH1-02-UA -> 732-5315-ND; MatesWith S9337-ND -> (none); NewDesigns YES -> (none); Package 2.54mm pin header -> (none); Stocked Bulk -> (none); Style THT -> (none)
- R12, R13: value R_499 -> R_500; footprint OEM:R_0603 -> Resistor_SMD:R_0603_1608Metric; symbol OEM:499R -> formula:R_500; DKPN 13-RC0603FR-10499RLDKR-ND -> (none); MFN Yageo -> DK; MPN RC0603FR-10499RL -> 541-3305-1-ND; NewDesigns YES -> (none); Package 0603 -> (none); PurchasingLink (none) -> https://www.digikey.com/en/products/detail/vishay-dale/TNPU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; Stocked Digi-Reel -> (none); Style SMD -> (none)
- R14: footprint OEM:R_0603 -> Resistor_SMD:R_0603_1608Metric; symbol OEM:120R -> formula:R_120; DKPN 13-RC0603FR-13120RLDKR-ND -> (none); MFN Yageo -> DK; MPN RC0603FR-13120RL -> 667-ERJ-6ENF1200V; NewDesigns YES -> (none); Package 0603 -> (none); PurchasingLink (none) -> https://www.mouser.com/ProductDetail/Panasonic-Industrial-D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; Stocked Digi-Reel -> (none); Style SMD -> (none)
- U4: symbol OEM:MCP25625-x-SS -> formula:MCP25625-x-SS; DKPN MCP25625T-E/SSCT-ND -> (none); MFN Microchip -> DK; MPN MCP25625 -> MCP25625-E/SS-ND; NewDesigns CHECK STOCK FIRST -> (none); Package SSOP-28 -> (none); PurchasingLink (none) -> https://www.digikey.com/product-detail/en/microchip-technol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; Stocked Tape -> (none); Style SMD -> (none)
- Y2: footprint OEM:Crystal_TXC7M -> footprints:Crystal_SMD_FA238; symbol OEM:Crystal_16MHz_18pF -> formula:Crystal_SMD; DKPN 887-1125-1-ND -> (none); MFN TXC -> DK; MPN 7M-16.000MAAJ-T -> 887-1125-1-ND; NewDesigns YES -> (none); Package Custom -> (none); PurchasingLink (none) -> https://www.digikey.com/product-detail/en/txc-corporation/7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; Stocked Tape -> (none); Style SMD -> (none)
Connections:
- net CAN_+ renamed CHARGER_CAN_+
- net CAN_- renamed CHARGER_CAN_-
- net MISO renamed MISO_CAN
- net MOSI renamed MOSI_CAN
- net SCK renamed SCK_CAN
