File: vehicle/mkvi/hardware/charging-cart/J1772/J1772.kicad_pcb (KiCad board)
At the start: 2 copper layers, 86.4 x 58.4 mm, 75 parts, among them J1 MicroFit_V_2, J2 MicroFit_V_2, J3 CONN_02x03, J4 CONN_01x02, J5 CONN_01x02, Q1 SSM3K333R, U1 ATmega328P-AU, U2 TLV70450DBVR, U3 MicroFit_VT_6, Y1 Crystal_16MHz_18pF

Commit message: Updating branch.
Parts:
- removed QR*****: hw.oem.to/J1772_1, OEM:QR_J1772_1
- removed the REF** at (92.8, 87.0)
- removed kibuzzard-63BF4696: G***, kibuzzard-63BF4696
- removed kibuzzard-63D45B3E: G***, kibuzzard-63D45B3E
- removed kibuzzard-63D45B6F: G***, kibuzzard-63D45B6F
- removed kibuzzard-63D83171: G***, kibuzzard-63D83171
- removed kibuzzard-63D8317A: G***, kibuzzard-63D8317A
- removed kibuzzard-63D831AC: G***, kibuzzard-63D831AC
- C1, C2, C7, C8: footprint OEM:C_0603 -> Capacitor_SMD:C_0603_1608Metric
- C10, C11, C14, C15, C16, C9: value 0.1uF -> C_0.1uF; footprint OEM:C_0603 -> footprints:C_0805_OEM
- C12, C13, C17, C18: footprint OEM:C_0603 -> footprints:C_0805_OEM
- C3, C5, C6: value 0.1uF -> C_0.1uF; footprint OEM:C_0603 -> Capacitor_SMD:C_0603_1608Metric
- C4: footprint OEM:C_0603 -> footprints:C_0603_1608Metric
- D1: value WHITE -> LED_0805_Red; footprint OEM:CHIPLED_0805 -> footprints:LED_0805_OEM
- D2, D4, D5: value WHITE -> LED_0805; footprint OEM:CHIPLED_0805 -> footprints:LED_0805_OEM
- D3: value SMBJ5355B-TP -> D_Zener_18V
- J3: value CONN_02x03 -> CONN_02X03
- Q1: footprint OEM:SOT-23F -> footprints:SOT-23F
- R1, R14, R17, R2, R3, R4, R5, R6, R7, R8, R9: footprint OEM:R_0603 -> Resistor_SMD:R_0603_1608Metric
- R10: value 1KR -> R_200; footprint OEM:R_0603 -> Resistor_SMD:R_0603_1608Metric
- R11: footprint Resistor_SMD:R_2512_6332Metric -> footprints:R_2512_OEM
- R12, R13, R15, R16: value R_499 -> R_500; footprint OEM:R_0603 -> Resistor_SMD:R_0603_1608Metric
- U2: value TLV70450DBVR -> AP7370; footprint OEM:SOT-23-5 -> footprints:SOT-23-5
- Y1: value Crystal_16MHz_18pF -> Crystal_SMD; footprint OEM:Crystal_TXC7M -> footprints:Crystal_SMD_FA238
- Y2, Y3: footprint OEM:Crystal_TXC7M -> footprints:Crystal_SMD_FA238
- moved C7 4.90 mm to (89.1, 135.2), turned to 180 degrees
- moved C8 3.33 mm to (85.0, 129.6)
- moved Q1 0.62 mm to (158.0, 91.0), turned to 90 degrees
- moved Y2 0.06 mm to (128.5, 130.0)
Connections:
- Q1 pad 2: Net-(J2-Pad1) -> /control_pilot
- Q1 pad 3: /control_pilot -> Net-(J2-Pad1)
- U2 pad 1: GND -> +12V
- U2 pad 2: +12V -> GND
- U2 pad 3: Net-(C8-Pad1) -> (no net)
- U2 pad 5: (no net) -> Net-(C8-Pad1)
Routing:
- net +12V: track 25.5 -> 28.2 mm
- net Net-(J2-Pad1): track 25.6 -> 23.8 mm
- net Net-(C8-Pad1): track 20.4 -> 21.8 mm
- net /control_pilot: track 15.0 -> 14.1 mm
- net Net-(C12-Pad2): track 6.94 -> 6.19 mm
- net GND: track 61.2 -> 61.9 mm
- removed copper zone on F.Cu, net (none)
