File: vehicle/mkvi/hardware/charging-cart/J1772/J1772.kicad_sch (KiCad schematic)
At the start: 39 parts, among them J1 MicroFit_V_2, J2 MicroFit_V_2, J3 CONN_02x03, Q1 SSM3K333R, U1 ATmega328P-AU, U2 TLV70450DBVR, U3 MicroFit_VT_6, Y1 Crystal_16MHz_18pF

Commit message: Updating branch.
Parts:
- C1, C2: footprint OEM:C_0603 -> Capacitor_SMD:C_0603_1608Metric; symbol OEM:30pF -> formula:C_30pF; DKPN 738-CML0603C0G300JT50VDKR-ND -> (none); MFN Stackpole Electronics -> DK; MPN CML0603C0G300JT50V -> 1276-1130-1-ND; NewDesigns YES -> (none); Package 0603 -> (none); PurchasingLink (none) -> https://www.digikey.com/product-detail/en/samsung-electro-m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; Stocked Digi-Reel -> (none); Style SMD -> (none)
- C3, C5, C6: value 0.1uF -> C_0.1uF; footprint OEM:C_0603 -> Capacitor_SMD:C_0603_1608Metric; symbol OEM:0u1F -> formula:C_0.1uF; DKPN 1276-1935-2-ND -> (none); MFN Samsung Electro-Mechanics -> DK; MPN CL10B104KB8NNWC -> 478-3352-1-ND; NewDesigns YES -> (none); Package 0603 -> (none); PurchasingLink (none) -> https://www.digikey.com/products/en?keywords=478-3352-1-ND; Stocked Reel -> (none); Style SMD -> (none)
- C4: footprint OEM:C_0603 -> footprints:C_0603_1608Metric; symbol OEM:0u1F -> formula:C_100nF; DKPN 1276-1935-2-ND -> (none); MFN Samsung Electro-Mechanics -> DK; MPN CL10B104KB8NNWC -> 1276-6717-1-ND; NewDesigns YES -> (none); Package 0603 -> (none); PurchasingLink (none) -> https://www.digikey.com/product-detail/en/samsung-electro-m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; Stocked Reel -> (none); Style SMD -> (none)
- C7, C8: footprint OEM:C_0603 -> Capacitor_SMD:C_0603_1608Metric; symbol OEM:1uF -> formula:C_1uF; DKPN 1276-1184-2-ND -> (none); MFN Samsung Electro-Mechanics -> DK; MPN CL10B105KA8NNNC -> 1276-6470-1-ND; NewDesigns YES -> (none); Package 0603 -> (none); PurchasingLink (none) -> https://www.digikey.com/en/products/detail/samsung-electro-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; Stocked Reel -> (none); Style SMD -> (none)
- D1: value WHITE -> LED_0805_Red; footprint OEM:CHIPLED_0805 -> footprints:LED_0805_OEM; symbol OEM:LED_WHITE -> formula:LED_0805_Red; DKPN 3147-B1701TW--20P000314U1930DKR-ND -> (none); MFN Harvatek -> DK; MPN B1701TW--20P000314U1930 -> 475-1415-1-ND; NewDesigns Yes -> (none); Package 0805 -> (none); PurchasingLink (none) -> https://www.digikey.com/product-detail/en/osram-opto-semico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; Stocked Digi-Reel -> (none); Style SMD -> (none)
- D2, D4, D5: value WHITE -> LED_0805; footprint OEM:CHIPLED_0805 -> footprints:LED_0805_OEM; symbol OEM:LED_WHITE -> formula:LED_0805; DKPN 3147-B1701TW--20P000314U1930DKR-ND -> (none); MFN Harvatek -> DK; MPN B1701TW--20P000314U1930 -> 475-1410-1-ND; NewDesigns Yes -> (none); Package 0805 -> (none); PurchasingLink (none) -> https://www.digikey.com/products/en?keywords=475-1410-1-ND; Stocked Digi-Reel -> (none); Style SMD -> (none)
- D3: value SMBJ5355B-TP -> D_Zener_18V; symbol OEM:SMBJ5355B-TP -> formula:D_Zener_18V; DKPN SMBJ5355B-TPMSCT-ND -> (none); MFN Micro Commercial Co -> DK; MPN SMBJ5355B-TP -> SMBJ5355B-TPMSCT-ND; NewDesigns YES -> (none); Package DO-214AA -> (none); PurchasingLink (none) -> https://www.digikey.com/products/en?keywords=SMBJ5355B-TPMS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; Stocked Tape -> (none); Style SMD -> (none)
- F1: symbol OEM:F_500mA_16V -> formula:F_500mA_16V; DKPN 507-1786-1-ND -> (none); MFN Bel Fuse -> DK; MPN 0ZCH0050FF2G -> 507-1786-1-ND; NewDesigns YES -> (none); Package 1210 -> (none); PurchasingLink (none) -> https://www.digikey.com/product-detail/en/bel-fuse-inc/0ZCH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; Stocked Tape -> (none); Style SMD -> (none)
- J1, J2: symbol OEM:MicroFit_VT_2 -> formula:MicroFit_V_2; DK (none) -> MFN; DKPN WM1789-ND -> (none); MFN Molex -> (none); MPN 0430450212 -> WM10660-ND; MatesWith 0430250200 -> (none); NewDesigns YES -> (none); Package Custom -> (none); PurchasingLink (none) -> https://www.digikey.com/product-detail/en/molex/0430450225/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; Stocked Tray -> (none); Style THT -> (none)
- J3: value CONN_02x03 -> CONN_02X03; symbol OEM:CONN_02x03 -> formula:CONN_02X03; DKPN 10129381-906002BLF-ND -> (none); MFN Ampehnol ICC -> DK; MPN 10129381-906002BLF -> 609-3234-ND; NewDesigns YES -> (none); Package .1" pin header -> (none); PurchasingLink (none) -> https://www.digikey.com/product-detail/en/amphenol-fci/6799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; Stocked Bulk -> (none); Style THT -> (none)
- Q1: footprint OEM:SOT-23F -> footprints:SOT-23F; symbol OEM:SSM3K333R -> formula:SSM3K333R; DKPN SSM3K333RLFDKR-ND -> (none); MFN Toshiba -> DK; MPN SSM3K333R,LF -> SSM3K333RLFCT-ND; NewDesigns YES -> (none); Package SOT-23 -> (none); PurchasingLink (none) -> https://www.digikey.com/product-detail/en/toshiba-semicondu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; Stocked Digi-Reel -> (none); Style SMD -> (none)
- R1: footprint OEM:R_0603 -> Resistor_SMD:R_0603_1608Metric; symbol OEM:10KR -> formula:R_10K; DKPN RMCF0603FT10K0TR-ND -> (none); MFN Stackpole Electronics -> DK; MPN RMCF0603FT10K0 -> CRS0805-FX-1002ELFCT-ND; NewDesigns YES -> (none); Package 0603 -> (none); PurchasingLink (none) -> https://www.digikey.com/products/en?keywords=CRS0805-FX-100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; Stocked Reel -> (none); Style SMD -> (none)
- R10: value 1KR -> R_200; footprint OEM:R_0603 -> Resistor_SMD:R_0603_1608Metric; symbol OEM:1KR -> formula:R_200; DKPN RMCF0603FT1K00TR-ND -> (none); MFN Stackpole Electronics -> DK; MPN RMCF0603FT1K00 -> RMCF0805JT200RCT-ND; NewDesigns YES -> (none); Package 0603 -> (none); Stocked Reel -> (none); Style SMD -> (none)
- R11: footprint Resistor_SMD:R_2512_6332Metric -> footprints:R_2512_OEM; symbol OEM:0R_2512 -> formula:R_0_2512; DKPN CR2512-J/-000ELFCT-ND -> (none); MFN Stackpole Electronics -> DK; MPN CR2512-J/-000ELF -> A121322CT-ND; NewDesigns YES -> (none); Package 2512 -> (none); PurchasingLink (none) -> https://www.digikey.com/products/en?keywords=A121322CT-ND; Stocked Tape -> (none); Style SMD -> (none)
- R2, R3, R9: footprint OEM:R_0603 -> Resistor_SMD:R_0603_1608Metric; symbol OEM:1KR -> formula:R_1K; DKPN RMCF0603FT1K00TR-ND -> (none); MFN Stackpole Electronics -> DK; MPN RMCF0603FT1K00 -> RNCP0805FTD1K00CT-ND; NewDesigns YES -> (none); Package 0603 -> (none); PurchasingLink (none) -> https://www.digikey.com/products/en?keywords=RNCP0805FTD1K0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; Stocked Reel -> (none); Style SMD -> (none)
- R4: footprint OEM:R_0603 -> Resistor_SMD:R_0603_1608Metric; symbol OEM:3KR -> formula:R_1K; DKPN 13-RC0603FR-103KLDKR-ND -> (none); MFN Yageo -> DK; MPN RC0603FR-103KL -> RNCP0805FTD1K00CT-ND; NewDesigns YES -> (none); Package 0603 -> (none); PurchasingLink (none) -> https://www.digikey.com/products/en?keywords=RNCP0805FTD1K0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; Stocked Digi-Reel -> (none); Style SMD -> (none)
- R5: footprint OEM:R_0603 -> Resistor_SMD:R_0603_1608Metric; symbol OEM:330R -> formula:R_330; DKPN 1292-WR06X3300FTLDKR-ND -> (none); MFN Walsin -> DK; MPN WR06X3300FTL -> RMCF0805FT330RCT-ND; NewDesigns YES -> (none); Package 0603 -> (none); PurchasingLink (none) -> https://www.digikey.com/product-detail/en/stackpole-electro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; Stocked Digi-Reel -> (none); Style SMD -> (none)
- R6: footprint OEM:R_0603 -> Resistor_SMD:R_0603_1608Metric; symbol OEM:2K2R -> formula:R_2.2K; DKPN 1292-WR06X222JTLDKR-ND -> (none); MFN Walsin Technology -> DK; MPN WR06X222 JTL -> RMCF0805FT2K20CT-ND; NewDesigns YES -> (none); Package 0603 -> (none); PurchasingLink (none) -> https://www.digikey.com/product-detail/en/stackpole-electro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; Stocked Digi-Reel -> (none); Style SMD -> (none)
- R7: footprint OEM:R_0603 -> Resistor_SMD:R_0603_1608Metric; symbol OEM:1K43R -> formula:R_1.43K; DKPN RMCF0603FT1K43DKR-ND -> (none); MFN Stackpole Electronics -> DK; MPN RMCF0603FT1K43 -> A103351CT-ND; NewDesigns YES -> (none); Package 0603 -> (none); PurchasingLink (none) -> https://www.digikey.com/product-detail/en/te-connectivity-p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; Stocked Digi-Reel -> (none); Style SMD -> (none)
- R8: footprint OEM:R_0603 -> Resistor_SMD:R_0603_1608Metric; symbol OEM:1K91R -> formula:R_1.91K; DKPN RMCF0603FT1K91DKR-ND -> (none); MFN Stackpole Electronics -> DK; MPN RMCF0603FT1K91 -> RNCF0805DTE1K91CT-ND; NewDesigns YES -> (none); Package 0603 -> (none); PurchasingLink (none) -> https://www.digikey.com/en/products/detail/stackpole-electr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; Stocked Digi-Reel -> (none); Style SMD -> (none)
- TP1, TP2, TP3, TP4: symbol OEM:TP_SMD -> formula:TP; DKPN 36-5019TR-ND -> (none); MFN Keystone -> DK; MPN 5019 -> 36-5006-ND; NewDesigns YES -> (none); Package Custom -> (none); PurchasingLink (none) -> https://www.digikey.com/product-detail/en/keystone-electron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; Stocked Reel -> (none); Style SMD -> (none)
- TP5, TP6: symbol OEM:TP_SMD -> formula:Test_Point_SMD; DKPN 36-5019TR-ND -> (none); MFN Keystone -> (none); MPN 5019 -> (none); NewDesigns YES -> (none); Package Custom -> (none); Stocked Reel -> (none); Style SMD -> (none)
- U1: symbol OEM:ATMEGA328P-AU -> formula:ATmega328P-AU; DKPN SAMPLE -> (none); MFN Microchip -> DK; MPN ATMEGA328P-AU -> ATMEGA328P-15AZTR-ND; NewDesigns No -> (none); Package 32-TQFP -> (none); PurchasingLink (none) -> https://www.digikey.com/product-detail/en/microchip-technol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; Stocked No -> (none); Style SMD -> (none)
- U2: value TLV70450DBVR -> AP7370; footprint OEM:SOT-23-5 -> footprints:SOT-23-5; symbol OEM:TLV70450DBVR -> formula:AP7370; DKPN 296-39287-1-ND -> (none); MFN STMicroelectronics -> DK; MPN TLV70450DBVR -> AP7370-50W5-7DICT-ND; NewDesigns YES -> (none); Package SOT23-5 -> (none); PurchasingLink (none) -> https://www.digikey.com/en/products/detail/diodes-incorpora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; Stocked Tape -> (none); Style SMD -> (none)
- U3: symbol OEM:MicroFit_VT_3x2 -> formula:MicroFit_VT_6; DKPN WM1797-ND -> (none); MFN Molex -> (none); NewDesigns YES -> (none); Package Custom -> (none); PurchasingLink (none) -> https://www.digikey.com/product-detail/en/molex/0430450614/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; Stocked Tray -> (none); Style THT -> (none)
- Y1: value Crystal_16MHz_18pF -> Crystal_SMD; footprint OEM:Crystal_TXC7M -> footprints:Crystal_SMD_FA238; symbol OEM:Crystal_16MHz_18pF -> formula:Crystal_SMD; DKPN 887-1125-1-ND -> (none); MFN TXC -> DK; MPN 7M-16.000MAAJ-T -> 887-1125-1-ND; NewDesigns YES -> (none); Package Custom -> (none); PurchasingLink (none) -> https://www.digikey.com/product-detail/en/txc-corporation/7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; Stocked Tape -> (none); Style SMD -> (none)
Connections:
- net +12V: now also U2.1 (Vin); no longer U2.2 (VI)
- net GND: now also U2.2 (GND); no longer U2.1 (GND)
- net control_pilot: now also Q1.2 (S); no longer Q1.3 (D)
- net at J2.1, R8.1: now also Q1.3 (D); no longer Q1.2 (S)
- net at C8.1, F1.1: now also U2.5 (Vout); no longer U2.3 (VO)
