File: vehicle/mkvi/hardware/imu/imu.kicad_pcb (KiCad board)
At the start: 4 copper layers, 17 x 17 mm, 59 parts, among them J1 SMD_WIRE_TO_BOARD, J2 TagConnect_6, J3 SMD_WIRE_TO_BOARD, J4 SMD_WIRE_TO_BOARD, J5 SMD_WIRE_TO_BOARD, U1 MCP2561-E_SN, U2 ATMEGA16M1, U3 ICM-20948, U4 NCP718BMT500TBG, U5 NCP705MT18TCG, U6 TXB0104RUTR, Y1 Crystal_SMD

Commit message: Updating branch.
Parts:
- removed kibuzzard-647D6821: G***, kibuzzard-647D6821
- removed kibuzzard-647D6949: G***, kibuzzard-647D6949
- added TP5: TestPoint, footprints:TestPoint_Pad_D0.5mm, F.Cu at (118.0, 67.0)
- added TP9: TestPoint, footprints:TestPoint_Pad_D0.5mm, F.Cu at (121.2, 76.1)
- added kibuzzard-65FD3539: G***, kibuzzard-65FD3539, B.Cu at (121.9, 67.5)
- R4: value R_91 -> R_330
- moved TP8 0.89 mm to (118.4, 65.3)
- moved TP6 0.51 mm to (117.5, 66.3)
- moved TP12 0.22 mm to (118.4, 63.7)
- moved TP10 0.20 mm to (118.4, 64.5)
Connections:
- U2 pad 1: unconnected-(U2-Pad1) -> /MISO
- U2 pad 12: unconnected-(U2-Pad12) -> /SCK
- U2 pad 2: unconnected-(U2-Pad2) -> /MOSI
- U2 pad 28: /SCK -> /INT
- U2 pad 8: /MISO -> unconnected-(U2-(PCINT0/MISO/PSCOUT2A)PB0-Pad8)
- U2 pad 9: /MOSI -> unconnected-(U2-(PCINT1/MOSI/PSCOUT2B)PB1-Pad9)
- U3 pad 12: unconnected-(U3-Pad12) -> /INT
- U4 pad : (no net) -> GND
- U5 pad : (no net) -> GND
- U6 pad 12: +5V -> +1V8
Routing:
- net +5V: track 28.7 -> 38.1 mm
- net /INT: track 0.00 -> 7.28 mm, vias 0 -> 2
- net /SCK: track 30.0 -> 23.7 mm
- net GND: track 37.0 -> 41.3 mm, vias 10 -> 11
- net /MISO: track 19.0 -> 22.9 mm
- net /MOSI: track 25.6 -> 27.7 mm, vias 2 -> 3
- net /CS: track 21.5 -> 20.5 mm
- net Net-(D1-K): track 3.40 -> 2.48 mm
- net +1V8: track 22.3 -> 22.9 mm
- net Net-(U3-REGOUT): track 5.50 -> 4.96 mm
Other:
- rule pad_to_mask_clearance: 0.051 -> 0
